File: Retro_Stereo_Main_Board/pcb_design/MCU-STM32H747BIT6.kicad_sch (KiCad schematic)
At the start: 42 parts, among them U1 STM32H747BITx

Commit message: Define crystals, add peripherals
Signed-off-by: Francisco <fran.testa07Qgmail.com>
Parts:
- added C49, C50, C51, C52: 33pF, symbol Device:C_Small
- added Y1: 12MHz, symbol Device:Crystal_GND24
- added Y2: 32.768kHz, symbol Device:Crystal
Connections:
- net GND: now also C49.2, C50.2, C51.2, C52.2, Y1.2 (G), Y1.4 (G)
- net at U1.11 (PC14): now also C52.1, Y2.2
- net at U1.12 (PC15): now also C51.1, Y2.1
- net TOUCH_SDA: now reaches U1.22 (PF0)
- net TOUCH_SCL: now reaches U1.23 (PF1)
- net TOUCH_RST: now reaches U1.24 (PF2)
- net TOUCH_INT: now reaches U1.25 (PF3)
- net at U1.35 (PH0): now also C49.1, Y1.1
- net at U1.36 (PH1): now also C50.1, Y1.3
- net DSIHOST_TE: no longer names the net of U1.88 (PB11)
- no-connect marks 93 -> 86

Commit message: Complete connections to display, add power block
Signed-off-by: Francisco <fran.testa07Qgmail.com>
Connections:
- net PMIC_CTRL: now reaches U1.131 (PG3)
- net VCI_EN: now reaches U1.134 (PG4)
- net VDDIO_EN: now reaches U1.135 (PG5)
- no-connect marks 86 -> 83
Changed lines of the file:
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@@
-	)
-	(no_connect
-		(at 163.83 181.61)
 	)
 	(no_connect
@@
 	)
 	(no_connect
-		(at 163.83 184.15)
-	)
-	(no_connect
 		(at 265.43 204.47)
 	)
@@
 	)
 	(no_connect
-		(at 163.83 179.07)
-	)
-	(no_connect
 		(at 265.43 194.31)
 	)
@@
 	(wire
 		(pts
+			(xy 129.54 184.15) (xy 163.83 184.15)
+		)
+		(stroke
+			(width 0)
+			(type default)
+		)
+	)
+	(wire
+		(pts
 			(xy 140.97 219.71) (xy 163.83 219.71)
 		)
@@
 	(wire
 		(pts
+			(xy 129.54 181.61) (xy 163.83 181.61)
+		)
+		(stroke
+			(width 0)
+			(type default)
+		)
+	)
+	(wire
+		(pts
 			(xy 21.59 83.82) (xy 21.59 85.09)
 		)
@@
 		(pts
 			(xy 265.43 80.01) (xy 290.83 80.01)
+		)
+		(stroke
+			(width 0)
+			(type default)
+		)
+	)
+	(wire
+		(pts
+			(xy 129.54 179.07) (xy 163.83 179.07)
 		)
 		(stroke
@@
 		)
 	)
+	(hierarchical_label "VDDIO_EN"
+		(shape output)
+		(at 129.54 184.15 180)
+		(effects
+			(font
+				(size 1.27 1.27)
+			)
+			(justify right)
+		)
+	)
 	(hierarchical_label "BTN_PREV"
 		(shape input)
@@
 		)
 	)
+	(hierarchical_label "PMIC_CTRL"
+		(shape output)
+		(at 129.54 179.07 180)
+		(effects
+			(font
+				(size 1.27 1.27)
+			)
+			(justify right)
+		)
+	)
 	(hierarchical_label "DSI_D0_-"
 		(shape output)
@@
 		(effects
 			(font
+				(size 1.27 1.27)
+			)
+			(justify right)
+		)
+	)
+	(hierarchical_label "VCI_EN"
+		(shape output)
+		(at 129.54 181.61 180)
+		(effects
+			(font

Commit message: Add Aux port interface
- Also add bluetooth interface IC

Signed-off-by: Francisco <fran.testa07Qgmail.com>
Connections:
- net NRST: now reaches C30.1, R1.2, U1.37 (NRST)
- net ENCODER_BTN: now reaches U1.81 (PE10)
- no-connect marks 83 -> 82
Other:
- moved on the sheet: C1, C16, C17, C18, C19, C2, C20, C22, C23, C24, C25, C26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

Commit message: Complete TEF6686 schematic page
- Start Bluetooth input design

Signed-off-by: Francisco <fran.testa07Qgmail.com>
Connections:
- net FM_GPIO_0: now reaches U1.26 (PF4)
- net FM_GPIO_1: now reaches U1.27 (PF5)
- net FM_GPIO_2: now reaches U1.30 (PF6)
- no-connect marks 82 -> 79
Changed lines of the file:
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@@
 	)
 	(no_connect
-		(at 163.83 224.79)
-	)
-	(no_connect
 		(at 265.43 105.41)
 	)
@@
 	)
 	(no_connect
-		(at 163.83 227.33)
-	)
-	(no_connect
 		(at 265.43 204.47)
 	)
 	(no_connect
-		(at 163.83 229.87)
-	)
-	(no_connect
 		(at 265.43 184.15)
 	)
@@
 	(wire
 		(pts
+			(xy 139.7 227.33) (xy 163.83 227.33)
+		)
+		(stroke
+			(width 0)
+			(type default)
+		)
+	)
+	(wire
+		(pts
 			(xy 294.64 38.1) (xy 294.64 39.37)
 		)
@@
 	(wire
 		(pts
+			(xy 139.7 229.87) (xy 163.83 229.87)
+		)
+		(stroke
+			(width 0)
+			(type default)
+		)
+	)
+	(wire
+		(pts
 			(xy 124.46 144.78) (xy 124.46 147.32)
 		)
@@
 	(wire
 		(pts
+			(xy 139.7 224.79) (xy 163.83 224.79)
+		)
+		(stroke
+			(width 0)
+			(type default)
+		)
+	)
+	(wire
+		(pts
 			(xy 163.83 262.89) (xy 160.02 262.89)
 		)
@@
 		)
 	)
+	(hierarchical_label "FM_GPIO_1"
+		(shape input)
+		(at 139.7 227.33 180)
+		(effects
+			(font
+				(size 1.27 1.27)
+			)
+			(justify right)
+		)
+	)
 	(hierarchical_label "BTN_SRC"
 		(shape input)
@@
 		)
 	)
+	(hierarchical_label "FM_GPIO_0"
+		(shape input)
+		(at 139.7 224.79 180)
+		(effects
+			(font
+				(size 1.27 1.27)
+			)
+			(justify right)
+		)
+	)
 	(hierarchical_label "SD_D1"
 		(shape input)
@@
 		)
 	)
+	(hierarchical_label "FM_GPIO_2"
+		(shape input)
+		(at 139.7 229.87 180)
+		(effects
+			(font
+				(size 1.27 1.27)
+			)
+			(justify right)
+		)
+	)

Commit message: Complete BT module sheet
Signed-off-by: Francisco <fran.testa07Qgmail.com>
Connections:
- net BT_UART_RTS: now reaches U1.138 (PG8)
- net BT_UART_TX: now reaches U1.142 (PC6)
- net BT_UART_RX: now reaches U1.143 (PC7)
- net BT_UART_CTS: now reaches U1.184 (PG13)
- no-connect marks 79 -> 75
Changed lines of the file:
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@@
 	)
 	(no_connect
-		(at 265.43 151.13)
-	)
-	(no_connect
 		(at 163.83 252.73)
 	)
@@
 	)
 	(no_connect
-		(at 163.83 191.77)
-	)
-	(no_connect
-		(at 163.83 204.47)
-	)
-	(no_connect
 		(at 265.43 143.51)
 	)
@@
 	)
 	(no_connect
-		(at 265.43 153.67)
-	)
-	(no_connect
 		(at 163.83 138.43)
 	)
@@
 	(wire
 		(pts
+			(xy 129.54 191.77) (xy 163.83 191.77)
+		)
+		(stroke
+			(width 0)
+			(type default)
+		)
+	)
+	(wire
+		(pts
 			(xy 191.77 36.83) (xy 191.77 39.37)
 		)
@@
 	(wire
 		(pts
+			(xy 265.43 151.13) (xy 290.83 151.13)
+		)
+		(stroke
+			(width 0)
+			(type default)
+		)
+	)
+	(wire
+		(pts
 			(xy 27.94 40.64) (xy 27.94 41.91)
 		)
@@
 	(wire
 		(pts
+			(xy 129.54 204.47) (xy 163.83 204.47)
+		)
+		(stroke
+			(width 0)
+			(type default)
+		)
+	)
+	(wire
+		(pts
 			(xy 160.02 260.35) (xy 163.83 260.35)
 		)
@@
 	(wire
 		(pts
+			(xy 265.43 153.67) (xy 290.83 153.67)
+		)
+		(stroke
+			(width 0)
+			(type default)
+		)
+	)
+	(wire
+		(pts
 			(xy 314.96 173.99) (xy 314.96 182.88)
 		)
@@
 		)
 	)
+	(hierarchical_label "BT_UART_RTS"
+		(shape output)
+		(at 129.54 191.77 180)
+		(effects
+			(font
+				(size 1.27 1.27)
+			)
+			(justify right)
+		)
+	)
 	(hierarchical_label "TOUCH_SDA"
 		(shape output)
@@
 		)
 	)
+	(hierarchical_label "BT_UART_TX"
+		(shape output)
+		(at 290.83 151.13 0)
+		(effects
+			(font
+				(size 1.27 1.27)
+			)
+			(justify left)
+		)
+	)
 	(hierarchical_label "BTN_CALL_TAKE"
 		(shape input)
@@
 		)
 	)
+	(hierarchical_label "BT_UART_RX"
+		(shape input)
+		(at 290.83 153.67 0)
+		(effects
+			(font
+				(size 1.27 1.27)
+			)
+			(justify left)
+		)
+	)
 	(hierarchical_label "OUT_I2S_SCK"
 		(shape output)
@@
 		)
 	)
+	(hierarchical_label "BT_UART_CTS"
+		(shape input)
+		(at 129.54 204.47 180)
+		(effects
+			(font
+				(size 1.27 1.27)
+			)
+			(justify right)
+		)
+	)

Commit message: Add jumper resistors
Signed-off-by: Francisco <fran.testa07Qgmail.com>
Connections:
- net BT_UART_INT: now reaches U1.146 (PA8)
- net BT_RST: now reaches U1.147 (PA9)
- net BT_MFB: now reaches U1.148 (PA10)
- no-connect marks 75 -> 72
Changed lines of the file:
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@@
-	)
-	(no_connect
-		(at 265.43 69.85)
 	)
 	(no_connect
@@
 	)
 	(no_connect
-		(at 265.43 72.39)
-	)
-	(no_connect
 		(at 163.83 143.51)
 	)
@@
 	)
 	(no_connect
-		(at 265.43 74.93)
-	)
-	(no_connect
 		(at 265.43 260.35)
 	)
@@
 	(wire
 		(pts
+			(xy 265.43 72.39) (xy 290.83 72.39)
+		)
+		(stroke
+			(width 0)
+			(type default)
+		)
+	)
+	(wire
+		(pts
 			(xy 290.83 212.09) (xy 265.43 212.09)
 		)
@@
 	(wire
 		(pts
+			(xy 290.83 69.85) (xy 265.43 69.85)
+		)
+		(stroke
+			(width 0)
+			(type default)
+		)
+	)
+	(wire
+		(pts
 			(xy 219.71 36.83) (xy 217.17 36.83)
 		)
@@
 		(pts
 			(xy 50.8 40.64) (xy 50.8 41.91)
+		)
+		(stroke
+			(width 0)
+			(type default)
+		)
+	)
+	(wire
+		(pts
+			(xy 265.43 74.93) (xy 290.83 74.93)
 		)
 		(stroke
@@
 		)
 	)
+	(hierarchical_label "BT_MFB"
+		(shape output)
+		(at 290.83 74.93 0)
+		(effects
+			(font
+				(size 1.27 1.27)
+			)
+			(justify left)
+		)
+	)
 	(hierarchical_label "I2C_SDA"
 		(shape output)
@@
 		)
 	)
+	(hierarchical_label "BT_UART_INT"
+		(shape input)
+		(at 290.83 69.85 0)
+		(effects
+			(font
+				(size 1.27 1.27)
+			)
+			(justify left)
+		)
+	)
 	(hierarchical_label "OUT_I2S_SD"
 		(shape input)
@@
 		(effects
 			(font
+				(size 1.27 1.27)
+			)
+			(justify left)
+		)
+	)
+	(hierarchical_label "BT_RST"
+		(shape output)
+		(at 290.83 72.39 0)
+		(effects
+			(font
